Commit message: Rename aeroarms joints

File: robots_description/models/aeroarms/arm.transmission.xacro (robot description, xacro)
@@ -2,11 +2,11 @@
 <robot xmlns:xacro="http://ros.org/wiki/xacro">
   <!-- Transmission macro -->
-  <xacro:macro name="side_x_to_y_transmission" params="side x y">
-    <transmission name="t_${side}_${x}_to_${y}">
+  <xacro:macro name="qside_x_transmission" params="side x">
+    <transmission name="t_${side}_${x}">
       <type>transmission_interface/SimpleTransmission</type>
-      <joint name="${side}_${x}_to_${y}">
+      <joint name="q${side}_${x}">
         <hardwareInterface>EffortJointInterface</hardwareInterface>
       </joint>
-      <actuator name="m_${side}_${x}_to_${y}">
+      <actuator name="m_${side}_${x}">
         <hardwareInterface>EffortJointInterface</hardwareInterface>
         <mechanicalReduction>1</mechanicalReduction>
@@ -15,12 +15,12 @@
   </xacro:macro>
   <!-- Left arm -->
-  <side_x_to_y_transmission side="left" x="multi" y="shoulder"/>
-  <side_x_to_y_transmission side="left" x="shoulder" y="upperarm"/>
-  <side_x_to_y_transmission side="left" x="upperarm" y="elbow"/>
-  <side_x_to_y_transmission side="left" x="elbow" y="forearm"/>
+  <qside_x_transmission side="1" x="1"/>
+  <qside_x_transmission side="1" x="2"/>
+  <qside_x_transmission side="1" x="3"/>
+  <qside_x_transmission side="1" x="4"/>
   <!-- Right arm -->
-  <side_x_to_y_transmission side="right" x="multi" y="shoulder"/>
-  <side_x_to_y_transmission side="right" x="shoulder" y="upperarm"/>
-  <side_x_to_y_transmission side="right" x="upperarm" y="elbow"/>
-  <side_x_to_y_transmission side="right" x="elbow" y="forearm"/>
+  <qside_x_transmission side="2" x="1"/>
+  <qside_x_transmission side="2" x="2"/>
+  <qside_x_transmission side="2" x="3"/>
+  <qside_x_transmission side="2" x="4"/>
 </robot>

File: robots_description/models/aeroarms/geometry.xacro (robot description, xacro)
@@ -110,5 +110,5 @@
     </collision>
   </link>
-  <joint name="left_multi_to_shoulder" type="revolute">
+  <joint name="q1_1" type="revolute">
     <!--origin xyz="200.781e-3 125.235e-3 -123.775e-3"/-->
     <origin xyz="50e-3 120e-3 10e-3"/>
@@ -138,5 +138,5 @@
     </collision>
   </link>
-  <joint name="left_shoulder_to_upperarm" type="revolute">
+  <joint name="q1_2" type="revolute">
     <origin xyz="0 25.9e-3 -30e-3"/>
     <parent link="left_shoulder"/>
@@ -165,5 +165,5 @@
     </collision>
   </link>
-  <joint name="left_upperarm_to_elbow" type="revolute">
+  <joint name="q1_3" type="revolute">
     <origin xyz="0 13e-3 -250e-3"/>
     <parent link="left_upperarm"/>
@@ -192,5 +192,5 @@
     </collision>
   </link>
-  <joint name="left_elbow_to_forearm" type="revolute">
+  <joint name="q1_4" type="revolute">
     <origin xyz="80.9e-3 -34.502e-3 0"/>
     <parent link="left_elbow"/>
@@ -221,5 +221,5 @@
     </collision>
   </link>
-  <joint name="left_forearm_to_wrist_pitch" type="revolute">
+  <joint name="q1_5" type="revolute">
     <origin xyz="185e-03 -2e-03 0" rpy="0 0 ${0.5*pi}"/>
     <parent link="left_forearm"/>
@@ -250,5 +250,5 @@
     </collision>
   </link>
-  <joint name="left_wrist_pitch_to_wrist_yaw" type="revolute">
+  <joint name="q1_6" type="revolute">
     <origin xyz="0 0 0" rpy="0 0 0"/>
     <parent link="left_wrist_pitch"/>
@@ -279,5 +279,5 @@
     </collision>
   </link>
-  <joint name="right_multi_to_shoulder" type="revolute">
+  <joint name="q2_1" type="revolute">
     <!--origin xyz="200.781e-3 -124.765e-3 -123.775e-3"/-->
     <origin xyz="50e-3 -120e-3 10e-3"/>
@@ -307,5 +307,5 @@
     </collision>
   </link>
-  <joint name="right_shoulder_to_upperarm" type="revolute">
+  <joint name="q2_2" type="revolute">
     <origin xyz="0 -25.9e-3 -30e-3"/>
     <parent link="right_shoulder"/>
@@ -334,5 +334,5 @@
     </collision>
   </link>
-  <joint name="right_upperarm_to_elbow" type="revolute">
+  <joint name="q2_3" type="revolute">
     <origin xyz="0 -13e-3 -250e-3"/>
     <parent link="right_upperarm"/>
@@ -361,5 +361,5 @@
     </collision>
   </link>
-  <joint name="right_elbow_to_forearm" type="revolute">
+  <joint name="q2_4" type="revolute">
     <origin xyz="80.9e-3 34.502e-3 0"/>
     <parent link="right_elbow"/>
@@ -390,5 +390,5 @@
     </collision>
   </link>
-  <joint name="right_forearm_to_wrist_pitch" type="revolute">
+  <joint name="q2_5" type="revolute">
     <origin xyz="185e-03 2e-03 0" rpy="0 0 ${0.5*pi}"/>
     <parent link="right_forearm"/>
@@ -419,5 +419,5 @@
     </collision>
   </link>
-  <joint name="right_wrist_pitch_to_wrist_yaw" type="revolute">
+  <joint name="q2_6" type="revolute">
     <origin xyz="0 0 0" rpy="0 0 0"/>
     <parent link="right_wrist_pitch"/>
