Commit message: Adapt models to Firmware v1.7.3

File: robots_description/models/aeroarms/model.xacro (robot description, xacro)
@@ -8,4 +8,6 @@
   <xacro:arg name='visual_material' default='DarkGrey' />
   <xacro:arg name='enable_mavlink_interface' default='true' />
+  <xacro:arg name='enable_gps_plugin' default='true' />
+  <xacro:arg name='gps_noise' default='true' />
   <xacro:arg name='enable_ground_truth' default='false' />
   <xacro:arg name='enable_logging' default='false' />
@@ -14,4 +16,12 @@
   <!-- Instantiate aeroarms "mechanics" -->
   <xacro:include filename="$(find robots_description)/models/aeroarms/geometry.xacro" />
+  <xacro:if value="$(arg enable_gps_plugin)">
+    <!-- Instantiate gps plugin. -->
+    <xacro:gps_plugin_macro
+      namespace="${namespace}"
+      gps_noise="$(arg gps_noise)"
+      >
+    </xacro:gps_plugin_macro>
+  </xacro:if>
   <xacro:if value="$(arg enable_mavlink_interface)">
   <!-- Instantiate mavlink telemetry interface. -->

File: robots_description/models/aeroarms_pendulum/model.xacro (robot description, xacro)
@@ -8,4 +8,6 @@
   <xacro:arg name='visual_material' default='DarkGrey' />
   <xacro:arg name='enable_mavlink_interface' default='true' />
+  <xacro:arg name='enable_gps_plugin' default='true' />
+  <xacro:arg name='gps_noise' default='true' />
   <xacro:arg name='enable_ground_truth' default='false' />
   <xacro:arg name='enable_logging' default='false' />
@@ -14,4 +16,12 @@
   <!-- Instantiate aeroarms "mechanics" -->
   <xacro:include filename="$(find robots_description)/models/aeroarms_pendulum/geometry.xacro" />
+  <xacro:if value="$(arg enable_gps_plugin)">
+    <!-- Instantiate gps plugin. -->
+    <xacro:gps_plugin_macro
+      namespace="${namespace}"
+      gps_noise="$(arg gps_noise)"
+      >
+    </xacro:gps_plugin_macro>
+  </xacro:if>
   <xacro:if value="$(arg enable_mavlink_interface)">
   <!-- Instantiate mavlink telemetry interface. -->

File: robots_description/models/iris/model.xacro (robot description, xacro)
@@ -8,4 +8,6 @@
   <xacro:arg name='visual_material' default='DarkGrey' />
   <xacro:arg name='enable_mavlink_interface' default='true' />
+  <xacro:arg name='enable_gps_plugin' default='true' />
+  <xacro:arg name='gps_noise' default='true' />
   <xacro:arg name='enable_ground_truth' default='false' />
   <xacro:arg name='enable_logging' default='false' />
@@ -14,4 +16,12 @@
   <!-- Instantiate iris "mechanics" -->
   <xacro:include filename="$(find robots_description)/models/iris/geometry.xacro" />
+  <xacro:if value="$(arg enable_gps_plugin)">
+    <!-- Instantiate gps plugin. -->
+    <xacro:gps_plugin_macro
+      namespace="${namespace}"
+      gps_noise="$(arg gps_noise)"
+      >
+    </xacro:gps_plugin_macro>
+  </xacro:if>
   <xacro:if value="$(arg enable_mavlink_interface)">
   <!-- Instantiate mavlink telemetry interface. -->

File: robots_description/models/mbzirc/model.xacro (robot description, xacro)
@@ -8,4 +8,6 @@
   <xacro:arg name='visual_material' default='DarkGrey' />
   <xacro:arg name='enable_mavlink_interface' default='true' />
+  <xacro:arg name='enable_gps_plugin' default='true' />
+  <xacro:arg name='gps_noise' default='true' />
   <xacro:arg name='enable_ground_truth' default='false' />
   <xacro:arg name='enable_logging' default='false' />
@@ -14,13 +16,21 @@
   <!-- Instantiate mbzirc "mechanics" -->
   <xacro:include filename="$(find robots_description)/models/mbzirc/geometry.xacro" />
+  <xacro:if value="$(arg enable_gps_plugin)">
+    <!-- Instantiate gps plugin. -->
+    <xacro:gps_plugin_macro
+      namespace="${namespace}"
+      gps_noise="$(arg gps_noise)"
+      >
+    </xacro:gps_plugin_macro>
+  </xacro:if>
   <xacro:if value="$(arg enable_mavlink_interface)">
-  <!-- Instantiate mavlink telemetry interface. -->
-  <xacro:mavlink_interface_macro
-    namespace="${namespace}"
-    imu_sub_topic="/imu"
-    mavlink_addr="$(arg mavlink_addr)"
-    mavlink_udp_port="$(arg mavlink_udp_port)"
-    >
-  </xacro:mavlink_interface_macro>
+    <!-- Instantiate mavlink telemetry interface. -->
+    <xacro:mavlink_interface_macro
+      namespace="${namespace}"
+      imu_sub_topic="/imu"
+      mavlink_addr="$(arg mavlink_addr)"
+      mavlink_udp_port="$(arg mavlink_udp_port)"
+      >
+    </xacro:mavlink_interface_macro>
   </xacro:if>
   <!-- Mount an ADIS16448 IMU. -->

File: robots_description/urdf/component_snippets.xacro (robot description, xacro)
@@ -118,4 +118,13 @@
     </gazebo>
   </xacro:macro>
+  <!-- Macro to add the gps plugin. -->
+  <xacro:macro name="gps_plugin_macro" params="namespace gps_noise">
+    <gazebo>
+      <plugin name='gps_plugin' filename='libgazebo_gps_plugin.so'>
+        <robotNamespace>${namespace}</robotNamespace>
+        <gpsNoise>${gps_noise}</gpsNoise>
+      </plugin>
+    </gazebo>
+  </xacro:macro>
   <!-- Macro to add the mavlink interface. -->
   <xacro:macro name="mavlink_interface_macro" params="namespace imu_sub_topic mavlink_addr mavlink_udp_port">
@@ -124,4 +133,5 @@
         <robotNamespace>${namespace}</robotNamespace>
         <imuSubTopic>${imu_sub_topic}</imuSubTopic>
+        <gpsSubTopic>/gps</gpsSubTopic>
         <mavlink_addr>$(arg mavlink_addr)</mavlink_addr>
         <mavlink_udp_port>$(arg mavlink_udp_port)</mavlink_udp_port>
