Commit message: Add friction to joints

File: robots_description/models/aeroarms/geometry.xacro (robot description, xacro)
@@ -104,5 +104,5 @@
     <child link="left_shoulder"/>
     <axis xyz="0 0 1"/>
-    <dynamics damping="0.7" friction="0.0"/>
+    <dynamics damping="0.7" friction="0.4"/>
     <limit effort="5000.0" lower="${-0.5*pi}" upper="${0.5*pi}" velocity="1"/>
   </joint>
@@ -131,5 +131,5 @@
     <child link="left_upperarm"/>
     <axis xyz="0 1 0"/>
-    <dynamics damping="0.7" friction="0.0"/>
+    <dynamics damping="0.7" friction="0.4"/>
     <limit effort="5000.0" lower="${-0.5*pi}" upper="${0.5*pi}" velocity="1"/>
   </joint>
@@ -158,5 +158,5 @@
     <child link="left_elbow"/>
     <axis xyz="0 1 0"/>
-    <dynamics damping="0.7" friction="0.0"/>
+    <dynamics damping="0.7" friction="0.4"/>
     <limit effort="5000.0" lower="${-0.5*pi}" upper="${0.5*pi}" velocity="1"/>
   </joint>
@@ -185,5 +185,5 @@
     <child link="left_forearm"/>
     <axis xyz="1 0 0"/>
-    <dynamics damping="0.7" friction="0.0"/>
+    <dynamics damping="0.7" friction="0.4"/>
     <limit effort="5000.0" lower="${-0.5*pi}" upper="${0.5*pi}" velocity="1"/>
   </joint>
@@ -215,5 +215,5 @@
     <child link="right_shoulder"/>
     <axis xyz="0 0 1"/>
-    <dynamics damping="0.7" friction="0.0"/>
+    <dynamics damping="0.7" friction="0.4"/>
     <limit effort="5000.0" lower="${-0.5*pi}" upper="${0.5*pi}" velocity="1"/>
   </joint>
@@ -242,5 +242,5 @@
     <child link="right_upperarm"/>
     <axis xyz="0 1 0"/>
-    <dynamics damping="0.7" friction="0.0"/>
+    <dynamics damping="0.7" friction="0.4"/>
     <limit effort="5000.0" lower="${-0.5*pi}" upper="${0.5*pi}" velocity="1"/>
   </joint>
@@ -269,5 +269,5 @@
     <child link="right_elbow"/>
     <axis xyz="0 1 0"/>
-    <dynamics damping="0.7" friction="0.0"/>
+    <dynamics damping="0.7" friction="0.4"/>
     <limit effort="5000.0" lower="${-0.5*pi}" upper="${0.5*pi}" velocity="1"/>
   </joint>
@@ -296,5 +296,5 @@
     <child link="right_forearm"/>
     <axis xyz="1 0 0"/>
-    <dynamics damping="0.7" friction="0.0"/>
+    <dynamics damping="0.7" friction="0.4"/>
     <limit effort="5000.0" lower="${-0.5*pi}" upper="${0.5*pi}" velocity="1"/>
   </joint>

Commit message: Solve cloud tf issues

File: robots_description/models/aeroarms/geometry.xacro (robot description, xacro)
@@ -77,4 +77,16 @@
     <origin xyz="0 0 -0.10" rpy="0 1.57 0" />
   </xacro:camera_macro>
+  <link name="camera_depth_base_link"></link>
+  <joint name="camera_depth_base_joint" type="fixed">
+    <origin xyz="0.4 0 0" rpy="0 0 0"/>
+    <parent link="base_link"/>
+    <child link="camera_depth_base_link"/>
+  </joint>
+  <link name="camera_depth_link"></link>
+  <joint name="camera_depth_joint" type="fixed">
+    <origin xyz="0 0 0" rpy="${-pi/2} 0 ${-pi/2} "/>
+    <parent link="camera_depth_base_link"/>
+    <child link="camera_depth_link"/>
+  </joint>
   <!-- Left arm -->
   <!-- Inertias are not symmetrical, can't use xacro -->

Commit message: Add wrist pitch and yaw

File: robots_description/models/aeroarms/geometry.xacro (robot description, xacro)
@@ -200,4 +200,62 @@
     <limit effort="5000.0" lower="${-0.5*pi}" upper="${0.5*pi}" velocity="1"/>
   </joint>
+  <link name="left_wrist_pitch">
+    <inertial>
+      <origin xyz="0 0 0"/>
+      <!--mass value="0.049"/>
+      <inertia ixx="6.73e-06" ixy="-2.83e-06" ixz="-5.16e-08" iyy="9.42e-05" iyz="1.62e-08" izz="9.58e-05"/-->
+      <mass value="0.1"/>
+      <inertia ixx="8.5833e-04" ixy="0" ixz="0" iyy="8.5833e-04" iyz="0" izz="5e-04"/>
+    </inertial>
+    <visual>
+      <origin xyz="0 -32e-03 0"/>
+      <geometry>
+        <mesh filename="package://robots_description/models/aeroarms/meshes/visual/left/wrist_pitch.dae" scale=".001 .001 .001"/>
+      </geometry>
+    </visual>
+    <collision>
+      <origin xyz="0 -32e-03 0"/>
+      <geometry>
+        <mesh filename="package://robots_description/models/aeroarms/meshes/collision/left/wrist_pitch.dae" scale=".001 .001 .001"/>
+      </geometry>
+    </collision>
+  </link>
+  <joint name="left_forearm_to_wrist_pitch" type="revolute">
+    <origin xyz="185e-03 -2e-03 0" rpy="0 0 ${0.5*pi}"/>
+    <parent link="left_forearm"/>
+    <child link="left_wrist_pitch"/>
+    <axis xyz="1 0 0"/>
+    <dynamics damping="0.7" friction="0.4"/>
+    <limit effort="5000.0" lower="${-0.5*pi}" upper="${0.5*pi}" velocity="1"/>
+  </joint>
+  <link name="left_wrist_yaw">
+    <inertial>
+      <origin xyz="0 0 0"/>
+      <!--mass value="0.049"/>
+      <inertia ixx="6.73e-06" ixy="-2.83e-06" ixz="-5.16e-08" iyy="9.42e-05" iyz="1.62e-08" izz="9.58e-05"/-->
+      <mass value="0.1"/>
+      <inertia ixx="8.5833e-04" ixy="0" ixz="0" iyy="8.5833e-04" iyz="0" izz="5e-04"/>
+    </inertial>
+    <visual>
+      <origin xyz="0 -45e-03 0" rpy="0 0 ${0.5*pi}"/>
+      <geometry>
+        <mesh filename="package://robots_description/models/aeroarms/meshes/visual/left/wrist_yaw.dae" scale=".001 .001 .001"/>
+      </geometry>
+    </visual>
+    <collision>
+      <origin xyz="0 -45e-03 0" rpy="0 0 ${0.5*pi}"/>
+      <geometry>
+        <mesh filename="package://robots_description/models/aeroarms/meshes/collision/left/wrist_yaw.dae" scale=".001 .001 .001"/>
+      </geometry>
+    </collision>
+  </link>
+  <joint name="left_wrist_pitch_to_wrist_yaw" type="revolute">
+    <origin xyz="0 0 0" rpy="0 0 0"/>
+    <parent link="left_wrist_pitch"/>
+    <child link="left_wrist_yaw"/>
+    <axis xyz="0 0 1"/>
+    <dynamics damping="0.7" friction="0.4"/>
+    <limit effort="5000.0" lower="${-0.5*pi}" upper="${0.5*pi}" velocity="1"/>
+  </joint>
   <!-- Right arm -->
   <!-- Inertias are not symmetrical, can't use xacro -->
@@ -308,4 +366,62 @@
     <child link="right_forearm"/>
     <axis xyz="1 0 0"/>
+    <dynamics damping="0.7" friction="0.4"/>
+    <limit effort="5000.0" lower="${-0.5*pi}" upper="${0.5*pi}" velocity="1"/>
+  </joint>
+  <link name="right_wrist_pitch">
+    <inertial>
+      <origin xyz="0 0 0"/>
+      <!--mass value="0.049"/>
+      <inertia ixx="6.73e-06" ixy="-2.83e-06" ixz="-5.16e-08" iyy="9.42e-05" iyz="1.62e-08" izz="9.58e-05"/-->
+      <mass value="0.1"/>
+      <inertia ixx="8.5833e-04" ixy="0" ixz="0" iyy="8.5833e-04" iyz="0" izz="5e-04"/>
+    </inertial>
+    <visual>
+      <origin xyz="0 -32e-03 0"/>
+      <geometry>
+        <mesh filename="package://robots_description/models/aeroarms/meshes/visual/right/wrist_pitch.dae" scale=".001 .001 .001"/>
+      </geometry>
+    </visual>
+    <collision>
+      <origin xyz="0 -32e-03 0"/>
+      <geometry>
+        <mesh filename="package://robots_description/models/aeroarms/meshes/collision/right/wrist_pitch.dae" scale=".001 .001 .001"/>
+      </geometry>
+    </collision>
+  </link>
+  <joint name="right_forearm_to_wrist_pitch" type="revolute">
+    <origin xyz="185e-03 2e-03 0" rpy="0 0 ${0.5*pi}"/>
+    <parent link="right_forearm"/>
+    <child link="right_wrist_pitch"/>
+    <axis xyz="1 0 0"/>
+    <dynamics damping="0.7" friction="0.4"/>
+    <limit effort="5000.0" lower="${-0.5*pi}" upper="${0.5*pi}" velocity="1"/>
+  </joint>
+  <link name="right_wrist_yaw">
+    <inertial>
+      <origin xyz="0 0 0"/>
+      <!--mass value="0.049"/>
+      <inertia ixx="6.73e-06" ixy="-2.83e-06" ixz="-5.16e-08" iyy="9.42e-05" iyz="1.62e-08" izz="9.58e-05"/-->
+      <mass value="0.1"/>
+      <inertia ixx="8.5833e-04" ixy="0" ixz="0" iyy="8.5833e-04" iyz="0" izz="5e-04"/>
+    </inertial>
+    <visual>
+      <origin xyz="0 -45e-03 0" rpy="0 0 ${0.5*pi}"/>
+      <geometry>
+        <mesh filename="package://robots_description/models/aeroarms/meshes/visual/right/wrist_yaw.dae" scale=".001 .001 .001"/>
+      </geometry>
+    </visual>
+    <collision>
+      <origin xyz="0 -45e-03 0" rpy="0 0 ${0.5*pi}"/>
+      <geometry>
+        <mesh filename="package://robots_description/models/aeroarms/meshes/collision/right/wrist_yaw.dae" scale=".001 .001 .001"/>
+      </geometry>
+    </collision>
+  </link>
+  <joint name="right_wrist_pitch_to_wrist_yaw" type="revolute">
+    <origin xyz="0 0 0" rpy="0 0 0"/>
+    <parent link="right_wrist_pitch"/>
+    <child link="right_wrist_yaw"/>
+    <axis xyz="0 0 1"/>
     <dynamics damping="0.7" friction="0.4"/>
     <limit effort="5000.0" lower="${-0.5*pi}" upper="${0.5*pi}" velocity="1"/>

Commit message: Set more realistic weight values to new links

File: robots_description/models/aeroarms/geometry.xacro (robot description, xacro)
@@ -205,5 +205,5 @@
       <!--mass value="0.049"/>
       <inertia ixx="6.73e-06" ixy="-2.83e-06" ixz="-5.16e-08" iyy="9.42e-05" iyz="1.62e-08" izz="9.58e-05"/-->
-      <mass value="0.1"/>
+      <mass value="0.021"/>
       <inertia ixx="8.5833e-04" ixy="0" ixz="0" iyy="8.5833e-04" iyz="0" izz="5e-04"/>
     </inertial>
@@ -234,5 +234,5 @@
       <!--mass value="0.049"/>
       <inertia ixx="6.73e-06" ixy="-2.83e-06" ixz="-5.16e-08" iyy="9.42e-05" iyz="1.62e-08" izz="9.58e-05"/-->
-      <mass value="0.1"/>
+      <mass value="0.041"/>
       <inertia ixx="8.5833e-04" ixy="0" ixz="0" iyy="8.5833e-04" iyz="0" izz="5e-04"/>
     </inertial>
@@ -374,5 +374,5 @@
       <!--mass value="0.049"/>
       <inertia ixx="6.73e-06" ixy="-2.83e-06" ixz="-5.16e-08" iyy="9.42e-05" iyz="1.62e-08" izz="9.58e-05"/-->
-      <mass value="0.1"/>
+      <mass value="0.021"/>
       <inertia ixx="8.5833e-04" ixy="0" ixz="0" iyy="8.5833e-04" iyz="0" izz="5e-04"/>
     </inertial>
@@ -403,5 +403,5 @@
       <!--mass value="0.049"/>
       <inertia ixx="6.73e-06" ixy="-2.83e-06" ixz="-5.16e-08" iyy="9.42e-05" iyz="1.62e-08" izz="9.58e-05"/-->
-      <mass value="0.1"/>
+      <mass value="0.041"/>
       <inertia ixx="8.5833e-04" ixy="0" ixz="0" iyy="8.5833e-04" iyz="0" izz="5e-04"/>
     </inertial>

Commit message: Match joint zero with real arm

File: robots_description/models/aeroarms/geometry.xacro (robot description, xacro)
@@ -166,10 +166,10 @@
   </link>
   <joint name="q1_3" type="revolute">
-    <origin xyz="0 13e-3 -250e-3"/>
+    <origin xyz="0 13e-3 -250e-3" rpy="0 ${0.5*pi} 0"/>
     <parent link="left_upperarm"/>
     <child link="left_elbow"/>
     <axis xyz="0 1 0"/>
     <dynamics damping="0.7" friction="0.4"/>
-    <limit effort="5000.0" lower="${-0.5*pi}" upper="${0.5*pi}" velocity="1"/>
+    <limit effort="5000.0" lower="${-pi}" upper="0" velocity="1"/>
   </joint>
   <link name="left_forearm">
@@ -335,10 +335,10 @@
   </link>
   <joint name="q2_3" type="revolute">
-    <origin xyz="0 -13e-3 -250e-3"/>
+    <origin xyz="0 -13e-3 -250e-3" rpy="0 ${0.5*pi} 0"/>
     <parent link="right_upperarm"/>
     <child link="right_elbow"/>
     <axis xyz="0 1 0"/>
     <dynamics damping="0.7" friction="0.4"/>
-    <limit effort="5000.0" lower="${-0.5*pi}" upper="${0.5*pi}" velocity="1"/>
+    <limit effort="5000.0" lower="${-pi}" upper="0" velocity="1"/>
   </joint>
   <link name="right_forearm">

Commit message: Add a collision mesh for multirotor_base

File: robots_description/models/aeroarms/geometry.xacro (robot description, xacro)
@@ -5,10 +5,9 @@
   <xacro:property name="namespace" value="" />
   <xacro:property name="rotor_velocity_slowdown_sim" value="10" />
-  <xacro:property name="mesh_file" value="multirotor.dae" />
+  <xacro:property name="visual_mesh" value="visual.dae" />
+  <xacro:property name="collision_mesh" value="collision.dae" />
   <xacro:property name="mesh_scale" value=".001 .001 .001"/>
   <xacro:property name="mesh_scale_prop" value=".001 .001 .001"/>
   <xacro:property name="mass" value="5.850" /> <!-- [kg] -->
-  <xacro:property name="body_width" value="0.8" /> <!-- [m] -->
-  <xacro:property name="body_height" value="0.6" /> <!-- [m] -->
   <xacro:property name="mass_rotor" value="0.005" /> <!-- [kg] -->
   <xacro:property name="rotor_offset_top" value="0.0" /> <!-- [m] -->
@@ -51,7 +50,6 @@
     robot_namespace="${namespace}"
     mass="${mass}"
-    body_width="${body_width}"
-    body_height="${body_height}"
-    mesh_file="${mesh_file}"
+    visual_mesh="${visual_mesh}"
+    collision_mesh="${collision_mesh}"
     mesh_scale="${mesh_scale}"
     color="DarkGrey"

File: robots_description/models/aeroarms_pendulum/geometry.xacro (robot description, xacro)
@@ -2,13 +2,12 @@
 <robot name="aeroarms" xmlns:xacro="http://ros.org/wiki/xacro">
   <!-- Properties -->
-  <xacro:property name="model_name" value="aeroarms" />
+  <xacro:property name="model_name" value="aeroarms_pendulum" />
   <xacro:property name="namespace" value="" />
   <xacro:property name="rotor_velocity_slowdown_sim" value="10" />
-  <xacro:property name="mesh_file" value="multirotor.dae" />
+  <xacro:property name="visual_mesh" value="visual.dae" />
+  <xacro:property name="collision_mesh" value="collision.dae" />
   <xacro:property name="mesh_scale" value=".001 .001 .001"/>
   <xacro:property name="mesh_scale_prop" value=".001 .001 .001"/>
   <xacro:property name="mass" value="5.850" /> <!-- [kg] -->
-  <xacro:property name="body_width" value="0.8" /> <!-- [m] -->
-  <xacro:property name="body_height" value="0.6" /> <!-- [m] -->
   <xacro:property name="mass_rotor" value="0.005" /> <!-- [kg] -->
   <xacro:property name="rotor_offset_top" value="0.0" /> <!-- [m] -->
@@ -51,7 +50,6 @@
     robot_namespace="${namespace}"
     mass="${mass}"
-    body_width="${body_width}"
-    body_height="${body_height}"
-    mesh_file="${mesh_file}"
+    visual_mesh="${visual_mesh}"
+    collision_mesh="${collision_mesh}"
     mesh_scale="${mesh_scale}"
     color="DarkGrey"

File: robots_description/models/iris/geometry.xacro (robot description, xacro)
@@ -5,10 +5,9 @@
   <xacro:property name="namespace" value="" />
   <xacro:property name="rotor_velocity_slowdown_sim" value="10" />
-  <xacro:property name="mesh_file" value="multirotor.dae" />
+  <xacro:property name="visual_mesh" value="visual.dae" />
+  <xacro:property name="collision_mesh" value="collision.dae" />
   <xacro:property name="mesh_scale" value="1 1 1"/>
   <xacro:property name="mesh_scale_prop" value="1 1 1"/>
   <xacro:property name="mass" value="1.5" /> <!-- [kg] -->
-  <xacro:property name="body_width" value="0.47" /> <!-- [m] -->
-  <xacro:property name="body_height" value="0.11" /> <!-- [m] -->
   <xacro:property name="mass_rotor" value="0.005" /> <!-- [kg] -->
   <xacro:property name="arm_length_front_x" value="0.13" /> <!-- [m] -->
@@ -48,7 +47,6 @@
     robot_namespace="${namespace}"
     mass="${mass}"
-    body_width="${body_width}"
-    body_height="${body_height}"
-    mesh_file="${mesh_file}"
+    visual_mesh="${visual_mesh}"
+    collision_mesh="${collision_mesh}"
     mesh_scale="${mesh_scale}"
     color="${color}"

File: robots_description/models/mbzirc/geometry.xacro (robot description, xacro)
@@ -5,10 +5,9 @@
   <xacro:property name="namespace" value="" />
   <xacro:property name="rotor_velocity_slowdown_sim" value="10" />
-  <xacro:property name="mesh_file" value="multirotor.dae" />
+  <xacro:property name="visual_mesh" value="visual.dae" />
+  <xacro:property name="collision_mesh" value="collision.dae" />
   <xacro:property name="mesh_scale" value=".001 .001 .001"/>
   <xacro:property name="mesh_scale_prop" value=".001 .001 .001"/>
   <xacro:property name="mass" value="5.850" /> <!-- [kg] -->
-  <xacro:property name="body_width" value="0.8" /> <!-- [m] -->
-  <xacro:property name="body_height" value="0.6" /> <!-- [m] -->
   <xacro:property name="mass_rotor" value="0.005" /> <!-- [kg] -->
   <xacro:property name="rotor_offset_top" value="0.0" /> <!-- [m] -->
@@ -49,7 +48,6 @@
     robot_namespace="${namespace}"
     mass="${mass}"
-    body_width="${body_width}"
-    body_height="${body_height}"
-    mesh_file="${mesh_file}"
+    visual_mesh="${visual_mesh}"
+    collision_mesh="${collision_mesh}"
     mesh_scale="${mesh_scale}"
     color="DarkGrey"

File: robots_description/urdf/multirotor_base.xacro (robot description, xacro)
@@ -19,5 +19,5 @@
   <!-- Main multirotor link -->
   <xacro:macro name="multirotor_base_macro"
-    params="model_name description_package:=robots_description robot_namespace mass body_width body_height mesh_file mesh_scale color *inertia">
+    params="model_name description_package:=robots_description robot_namespace mass visual_mesh collision_mesh mesh_scale color *inertia">
     <link name="base_link"></link>
     <joint name="base_joint" type="fixed">
@@ -35,7 +35,6 @@
         <origin xyz="0 0 0" rpy="0 0 0" />
         <geometry>
-          <mesh filename="package://${description_package}/models/${model_name}/meshes/${mesh_file}"
+          <mesh filename="package://${description_package}/models/${model_name}/meshes/${visual_mesh}"
             scale="${mesh_scale}" />
-          <!-- <box size="${body_width} ${body_width} ${body_height}"/> --> <!-- [m] [m] [m] -->
         </geometry>
       </visual>
@@ -43,7 +42,6 @@
         <origin xyz="0 0 0" rpy="0 0 0" />
         <geometry>
-        <!--mesh filename="package://${description_package}/TODO/models/${model_name}/meshes/${mesh_file}"
-            scale="${mesh_scale}" /-->
-          <box size="${body_width} ${body_width} ${body_height}" /> <!-- [m] [m] [m] -->
+        <mesh filename="package://${description_package}/models/${model_name}/meshes/${collision_mesh}"
+            scale="${mesh_scale}" />
         </geometry>
       </collision>
