Commit message: Fake pendulum arm inertias

File: robots_description/models/aeroarms_pendulum/geometry.xacro (robot description, xacro)
@@ -94,5 +94,5 @@
       <origin xyz="0 0 -0.017"/>
       <mass value="0.016"/>
-      <inertia ixx="1e-04" ixy="0" ixz="0" iyy="1e-04" iyz="0" izz="1e-04"/>
+      <inertia ixx="5e-04" ixy="0" ixz="0" iyy="5e-04" iyz="0" izz="5e-04"/>
     </inertial>
     <visual>
@@ -117,5 +117,5 @@
     <inertial>
       <origin xyz="0 0 -0.80"/>
-      <mass value="0.440"/>
+      <mass value="0.240"/>
       <inertia ixx="0.0667" ixy="0" ixz="0" iyy="0.066" iyz="0" izz="0.0011"/>
     </inertial>
@@ -138,5 +138,5 @@
     <child link="pendulum_shoulder"/>
     <axis xyz="0 1 0"/>
-    <dynamics damping="0.7" friction="0.4"/>
+    <dynamics damping="0.2" friction="0.1"/>
     <limit effort="5000.0" lower="${-0.5*pi}" upper="${0.5*pi}" velocity="6"/>
   </joint>
@@ -147,5 +147,5 @@
       <origin xyz="0 -0.022 0"/>
       <mass value="0.101"/>
-      <inertia ixx="4e-04" ixy="0" ixz="0" iyy="1e-04" iyz="0" izz="1e-04"/>
+      <inertia ixx="8e-04" ixy="0" ixz="0" iyy="5e-04" iyz="0" izz="5e-04"/>
     </inertial>
     <visual>
@@ -172,5 +172,5 @@
       <origin xyz="0 0 0.035"/>
       <mass value="0.121"/>
-      <inertia ixx="5e-04" ixy="0" ixz="0" iyy="5e-04" iyz="0" izz="1e-04"/>
+      <inertia ixx="9e-04" ixy="0" ixz="0" iyy="9e-04" iyz="0" izz="5e-04"/>
     </inertial>
     <visual>
@@ -199,5 +199,5 @@
       <origin xyz="0 0 0.034"/>
       <mass value="0.087"/>
-      <inertia ixx="3e-04" ixy="0" ixz="0" iyy="3e-04" iyz="0" izz="1e-04"/>
+      <inertia ixx="7e-04" ixy="0" ixz="0" iyy="7e-04" iyz="0" izz="5e-04"/>
     </inertial>
     <visual>
@@ -226,5 +226,5 @@
       <origin xyz="0 0 -0.125"/>
       <mass value="0.100"/>
-      <inertia ixx="1e-04" ixy="0" ixz="0" iyy="1e-04" iyz="0" izz="1e-04"/>
+      <inertia ixx="5e-04" ixy="0" ixz="0" iyy="5e-04" iyz="0" izz="5e-04"/>
     </inertial>
     <visual>
@@ -255,5 +255,5 @@
       <origin xyz="0 0.022 0"/>
       <mass value="0.101"/>
-      <inertia ixx="4e-04" ixy="0" ixz="0" iyy="1e-04" iyz="0" izz="1e-04"/>
+      <inertia ixx="8e-04" ixy="0" ixz="0" iyy="5e-04" iyz="0" izz="5e-04"/>
     </inertial>
     <visual>
@@ -280,5 +280,5 @@
       <origin xyz="0 0 0.035"/>
       <mass value="0.121"/>
-      <inertia ixx="5e-04" ixy="0" ixz="0" iyy="5e-04" iyz="0" izz="1e-04"/>
+      <inertia ixx="9e-04" ixy="0" ixz="0" iyy="9e-04" iyz="0" izz="5e-04"/>
     </inertial>
     <visual>
@@ -307,5 +307,5 @@
       <origin xyz="0 0 0.034"/>
       <mass value="0.087"/>
-      <inertia ixx="3e-04" ixy="0" ixz="0" iyy="3e-04" iyz="0" izz="1e-04"/>
+      <inertia ixx="8e-04" ixy="0" ixz="0" iyy="8e-04" iyz="0" izz="5e-04"/>
     </inertial>
     <visual>
@@ -334,5 +334,5 @@
       <origin xyz="0 0 -0.125"/>
       <mass value="0.100"/>
-      <inertia ixx="1e-04" ixy="0" ixz="0" iyy="1e-04" iyz="0" izz="1e-04"/>
+      <inertia ixx="5e-04" ixy="0" ixz="0" iyy="5e-04" iyz="0" izz="5e-04"/>
     </inertial>
     <visual>

Commit message: Change some physics parameters

File: robots_description/models/aeroarms_pendulum/geometry.xacro (robot description, xacro)
@@ -116,7 +116,7 @@
   <link name="pendulum_shoulder">
     <inertial>
-      <origin xyz="0 0 -0.80"/>
-      <mass value="0.240"/>
-      <inertia ixx="0.0667" ixy="0" ixz="0" iyy="0.066" iyz="0" izz="0.0011"/>
+      <origin xyz="0 0 -0.785"/>
+      <mass value="0.520"/>
+      <inertia ixx="0.0457" ixy="0" ixz="0" iyy="0.045" iyz="0" izz="0.0011"/>
     </inertial>
     <visual>
@@ -138,5 +138,5 @@
     <child link="pendulum_shoulder"/>
     <axis xyz="0 1 0"/>
-    <dynamics damping="0.2" friction="0.1"/>
+    <dynamics damping="0.05" friction="0.05"/>
     <limit effort="5000.0" lower="${-0.5*pi}" upper="${0.5*pi}" velocity="6"/>
   </joint>
@@ -224,7 +224,7 @@
   <link name="left_forearm">
     <inertial>
-      <origin xyz="0 0 -0.125"/>
-      <mass value="0.100"/>
-      <inertia ixx="5e-04" ixy="0" ixz="0" iyy="5e-04" iyz="0" izz="5e-04"/>
+      <origin xyz="0 0 -0.085"/>
+      <mass value="0.140"/>
+      <inertia ixx="8e-04" ixy="0" ixz="0" iyy="8e-04" iyz="0" izz="5e-04"/>
     </inertial>
     <visual>
@@ -332,7 +332,7 @@
   <link name="right_forearm">
     <inertial>
-      <origin xyz="0 0 -0.125"/>
-      <mass value="0.100"/>
-      <inertia ixx="5e-04" ixy="0" ixz="0" iyy="5e-04" iyz="0" izz="5e-04"/>
+      <origin xyz="0 0 -0.085"/>
+      <mass value="0.140"/>
+      <inertia ixx="8e-04" ixy="0" ixz="0" iyy="8e-04" iyz="0" izz="5e-04"/>
     </inertial>
     <visual>
