Commit message: Add simulated laser scanner to componet snippets

File: robots_description/urdf/component_snippets.xacro (robot description, xacro)
@@ -522,3 +522,68 @@
     </xacro:imu_plugin_macro>
   </xacro:macro>
+  <!-- Macro to add a laser scanner -->
+  <xacro:macro name="laser_scanner"
+    params="namespace id parent_link update_rate sample_count
+    angle_min angle_max range_min range_max range_res visualize:=false *origin">
+    <joint name="${namespace}/laser_${id}_joint" type="fixed">
+      <xacro:insert_block name="origin" />
+      <parent link="${parent_link}"/>
+      <child link="${namespace}/laser_${id}_link"/>
+    </joint>
+    <link name="${namespace}/laser_${id}_link">
+      <collision>
+        <origin xyz="0 0 0" rpy="0 0 0"/>
+        <geometry>
+          <cylinder length="0.03" radius="0.04" />
+        </geometry>
+      </collision>
+      <visual>
+        <origin xyz="0 0 0" rpy="0 0 0"/>
+        <geometry>
+          <cylinder length="0.03" radius="0.04" />
+        </geometry>
+      </visual>
+      <inertial>
+        <mass value="1e-5" />
+        <origin xyz="0 0 0" rpy="0 0 0"/>
+        <inertia ixx="1e-6" ixy="0" ixz="0" iyy="1e-6" iyz="0" izz="1e-6" />
+      </inertial>
+    </link>
+    <gazebo reference="${namespace}/laser_${id}_link">
+      <sensor type="ray" name="${namespace}_laser_${id}_sensor">
+        <pose>0 0 0 0 0 0</pose>
+        <visualize>${visualize}</visualize>
+        <update_rate>${update_rate}</update_rate>
+        <ray>
+          <scan>
+            <horizontal>
+              <samples>${sample_count}</samples>
+              <resolution>1</resolution>
+              <min_angle>${angle_min}</min_angle>
+              <max_angle>${angle_max}</max_angle>
+            </horizontal>
+          </scan>
+          <range>
+            <min>${range_min}</min>
+            <max>${range_max}</max>
+            <resolution>${range_res}</resolution>
+          </range>
+          <noise>
+            <type>gaussian</type>
+            <!-- Noise parameters based on published spec for Hokuyo laser
+                achieving "+-30mm" accuracy at range < 10m.  A mean of 0.0m and
+                stddev of 0.01m will put 99.7% of samples within 0.03m of the true
+                reading. -->
+            <mean>0.0</mean>
+            <stddev>0.01</stddev>
+          </noise>
+        </ray>
+        <plugin name="${namespace}_laser_${id}_controller" filename="libgazebo_ros_laser.so">
+          <robotNamespace>${namespace}</robotNamespace>
+          <topicName>scan_${id}</topicName>
+          <frameName>${namespace}/laser_${id}_link</frameName>
+        </plugin>
+      </sensor>
+    </gazebo>
+  </xacro:macro>
 </robot>

Commit message: Add options to customize mavlink and lidar plugins

File: robots_description/urdf/component_snippets.xacro (robot description, xacro)
@@ -141,5 +141,6 @@
   </xacro:macro>
   <!-- Macro to add the mavlink interface. -->
-  <xacro:macro name="mavlink_interface_macro" params="namespace imu_sub_topic mavlink_addr mavlink_tcp_port mavlink_udp_port">
+  <xacro:macro name="mavlink_interface_macro" params="namespace imu_sub_topic mavlink_addr mavlink_tcp_port mavlink_udp_port octo:=false">
+    <xacro:property name="is_octo" value="${octo}"/>
     <gazebo>
       <plugin name="mavlink_interface" filename="libgazebo_mavlink_interface.so">
@@ -216,31 +217,53 @@
             <joint_control_type>velocity</joint_control_type>
           </channel>
-          <channel name="rotor7">
-            <input_index>6</input_index>
-            <input_offset>0</input_offset>
-            <!-- joint limits [-0.524, 0.524] -->
-            <input_scaling>0.524</input_scaling>
-            <zero_position_disarmed>0</zero_position_disarmed>
-            <zero_position_armed>0</zero_position_armed>
-            <joint_control_type>position</joint_control_type>
-            <joint_name>zephyr_delta_wing::flap_right_joint</joint_name>
-            <joint_control_pid>
-              <p>10.0</p>
-              <i>0</i>
-              <d>0</d>
-              <iMax>0</iMax>
-              <iMin>0</iMin>
-              <cmdMax>20</cmdMax>
-              <cmdMin>-20</cmdMin>
-            </joint_control_pid>
-          </channel>
-          <channel name="rotor8">
-            <input_index>7</input_index>
-            <input_offset>0</input_offset>
-            <input_scaling>0.524</input_scaling>
-            <zero_position_disarmed>0</zero_position_disarmed>
-            <zero_position_armed>0</zero_position_armed>
-            <joint_control_type>position</joint_control_type>
-          </channel>
+          <!-- Add extra velocity outputs for rotors 7 and 8 -->
+          <xacro:if value="${is_octo}">
+            <channel name="rotor7">
+              <input_index>6</input_index>
+              <input_offset>0</input_offset>
+              <input_scaling>1000</input_scaling>
+              <zero_position_disarmed>0</zero_position_disarmed>
+              <zero_position_armed>100</zero_position_armed>
+              <joint_control_type>velocity</joint_control_type>
+            </channel>
+            <channel name="rotor8">
+              <input_index>7</input_index>
+              <input_offset>0</input_offset>
+              <input_scaling>1000</input_scaling>
+              <zero_position_disarmed>0</zero_position_disarmed>
+              <zero_position_armed>100</zero_position_armed>
+              <joint_control_type>velocity</joint_control_type>
+            </channel>
+          </xacro:if>
+          <!-- Else -->
+          <xacro:if value="${not is_octo}">
+            <channel name="rotor7">
+              <input_index>6</input_index>
+              <input_offset>0</input_offset>
+              <!-- joint limits [-0.524, 0.524] -->
+              <input_scaling>0.524</input_scaling>
+              <zero_position_disarmed>0</zero_position_disarmed>
+              <zero_position_armed>0</zero_position_armed>
+              <joint_control_type>position</joint_control_type>
+              <joint_name>zephyr_delta_wing::flap_right_joint</joint_name>
+              <joint_control_pid>
+                <p>10.0</p>
+                <i>0</i>
+                <d>0</d>
+                <iMax>0</iMax>
+                <iMin>0</iMin>
+                <cmdMax>20</cmdMax>
+                <cmdMin>-20</cmdMin>
+              </joint_control_pid>
+            </channel>
+            <channel name="rotor8">
+              <input_index>7</input_index>
+              <input_offset>0</input_offset>
+              <input_scaling>0.524</input_scaling>
+              <zero_position_disarmed>0</zero_position_disarmed>
+              <zero_position_armed>0</zero_position_armed>
+              <joint_control_type>position</joint_control_type>
+            </channel>
+          </xacro:if>
         </control_channels>
       </plugin>
@@ -555,5 +578,5 @@
   <xacro:macro name="laser_scanner"
     params="namespace id pub_topic tf parent_link update_rate sample_count
-    angle_min angle_max range_min range_max range_res visualize:=false *origin">
+    angle_min angle_max range_min range_max range_res visualize:=false *origin length:=0.03 radius:=0.04">
     <joint name="${namespace}/laser_${id}_joint" type="fixed">
       <xacro:insert_block name="origin" />
@@ -565,5 +588,5 @@
         <origin xyz="0 0 0" rpy="0 0 0"/>
         <geometry>
-          <cylinder length="0.03" radius="0.04" />
+          <cylinder length="${length}" radius="${radius}" />
         </geometry>
       </collision>
@@ -571,5 +594,5 @@
         <origin xyz="0 0 0" rpy="0 0 0"/>
         <geometry>
-          <cylinder length="0.03" radius="0.04" />
+          <cylinder length="${length}" radius="${radius}" />
         </geometry>
       </visual>

File: robots_description/urdf/multirotor_base.xacro (robot description, xacro)
@@ -19,9 +19,9 @@
   <!-- Main multirotor link -->
   <xacro:macro name="multirotor_base_macro"
-    params="model_name description_package:=robots_description robot_namespace mass body_width body_height height_offset:=0 mesh_file mesh_scale color *inertia">
-    <link name="base_link"></link>
+    params="model_name description_package:=robots_description robot_namespace robot_base_link:=base_link mass body_width body_height height_offset:=0 mesh_file mesh_scale color *inertia">
+    <link name="${robot_base_link}"></link>
     <joint name="base_joint" type="fixed">
       <origin xyz="0 0 0" rpy="0 0 0" />
-      <parent link="base_link" />
+      <parent link="${robot_base_link}" />
       <child link="base_link_inertia" />
     </joint>
